File: ESP8266_ESP-01_Breakout_2015-11-16.brd (EAGLE design)
At the start: 16.9 x 20.2 mm, 4 parts

Commit message: Updates
Parts:
- moved LEFT 0.76 mm to (2.09, 18.6)
- moved RIGHT 0.76 mm to (14.7, 18.6)
- moved C1 0.76 mm to (14.2, 4.39)
- moved ESP-01 0.76 mm to (6.26, 3.88)
Other:
- board text added: "Vcc"
- board text removed: "[ESP8266] ESP-01 Breakout"
