File: Power/USB_Micro_Power_to_lab_board_2015-12-26.sch (EAGLE design)
At the start: 9 parts, among them IC1 REG1117

Commit message: Upgrades
Small changes
Parts:
- added JP5: (no value), pinhead:PINHD-1X2
- R1: value 100 -> (none)
Connections:
- net GND: now also JP5.2
- net N$1: now also JP5.1
Other:
- moved on the sheet: F1, IC1, JP1, JP2, JP3, JP4, POWER, R1
